Commit message: script fast.py moves the robot

File: robot_description/urdf/robot_z.urdf (robot description, URDF)
Before this commit: robot parallel_robot, 20 links, 19 joints
Joints:
- joint bridge_2_to_platform: limit lower=-0.7 upper=0.7 effort=1000.0 velocity=0.5 -> lower=-1.5 upper=1.5 effort=1000.0 velocity=2.5
- joint up_4_to_shuttle_1: limit lower=-0.7 upper=0.7 effort=1000.0 velocity=0.5 -> lower=-1.5 upper=1.5 effort=1000.0 velocity=0.5
